File: keyboard-pcb-mk1.kicad_pcb (KiCad board)
At the start: 2 copper layers, 94 x 38.1 mm, 24 parts, among them SW1 SW_Push, U1 ATmega32U4-AU, Y1 16MHz

Commit message: versino final
Parts:
- moved C1 156.8 mm to (131.6, 127.7)
- moved C2 156.8 mm to (119.9, 110.1)
- moved C3 156.8 mm to (139.2, 115.0)
- moved C4 156.8 mm to (117.6, 124.1)
- moved C5 156.8 mm to (131.8, 105.1)
- moved C6 156.8 mm to (122.9, 105.1)
- moved C7 156.8 mm to (116.4, 117.9)
- moved D1 156.8 mm to (159.6, 106.7)
- moved D2 156.8 mm to (160.1, 126.1)
- moved D3 156.8 mm to (178.4, 106.8)
- moved MX1 156.8 mm to (151.5, 106.5)
- moved MX2 156.8 mm to (151.5, 125.5)
- moved MX3 156.8 mm to (170.6, 106.5)
- moved MX4 156.8 mm to (170.6, 125.5)
- moved R1 156.8 mm to (95.2, 109.6)
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Routing:
- net Net-(D4-Pad2): track 7.81 -> 8.45 mm
- net Net-(D3-Pad2): track 7.75 -> 8.40 mm
- net Net-(D2-Pad2): track 8.18 -> 8.79 mm
Other:
- outline, holes or cut-outs redrawn
- net class Default removed
- net class Power removed
- board text added: "The solksingt is real"
